File: SoftStarter/SoftStarter.kicad_pcb (KiCad board)
At the start: 2 copper layers, 100 x 100 mm, 72 parts, among them J1 Conn_01x04_Female, J2 Conn_01x03_Female, J3 Conn_01x02_Male, J4 JTAG, J5 Conn_01x02_Female, Q1 BT136-500, Q2 BT136-500, Q3 BT136-500, T1 Trafo_20P_1S, T2 Current Transformer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

Commit message: fim do esquema, revisado
Parts:
- R16: value 150R -> 390R
- R18, R20: value 56R -> 390R
- R19: value 56R -> 150R
- U1: value LM317_TO3 -> LM317_3PinPackage
- moved C7 515.4 mm to (499.8, 135.0), turned to 90 degrees
- moved Q3 492.8 mm to (499.8, 111.4), turned to 180 degrees
- moved C6 483.6 mm to (482.2, 137.0), turned to 90 degrees
- moved Q1 479.8 mm to (473.8, 112.4), turned to 180 degrees
- moved R23 476.0 mm to (494.4, 120.0), turned to 270 degrees
- moved R21 472.8 mm to (462.0, 124.2), turned to 270 degrees
- moved C5 472.4 mm to (467.6, 137.4), turned to 90 degrees
- moved U4 470.7 mm to (497.2, 146.0), turned to 90 degrees
- moved R17 469.4 mm to (494.4, 137.0), turned to 270 degrees
- moved R8 463.6 mm to (497.2, 150.0), turned to 270 degrees
- moved R22 459.0 mm to (476.6, 124.4), turned to 270 degrees
- moved U2 458.1 mm to (465.2, 148.6), turned to 90 degrees
- moved Q2 449.5 mm to (484.4, 112.4), turned to 180 degrees
- moved U3 446.2 mm to (479.8, 148.6), turned to 90 degrees
- moved R18 443.4 mm to (474.0, 97.8)
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Connections:
- net Net-(J2-Pad1) renamed /R_CARGA
- C6 pad 2: Net-(C6-Pad2) -> /S_CARGA
- C7 pad 2: Net-(C7-Pad2) -> /T_CARGA
- J1 pad 1: VAC -> /T
- J1 pad 2: VAC -> /S
- J1 pad 3: VAC -> /R
- J2 pad 2: Net-(C6-Pad2) -> /S_CARGA
- J2 pad 3: Net-(C7-Pad2) -> /T_CARGA
- Q1 pad 1: Net-(C5-Pad2) -> /T_CARGA
- Q1 pad 2: VAC -> /T
- Q2 pad 1: Net-(C6-Pad2) -> Net-(C5-Pad2)
- Q2 pad 2: VAC -> /R
- Q3 pad 1: Net-(C7-Pad2) -> /S_CARGA
- Q3 pad 2: VAC -> /S
- R11 pad 2: VAC -> /S
- R13 pad 2: VAC -> /T
- R16 pad 1: Net-(C6-Pad1) -> Net-(C5-Pad2)
- R16 pad 2: Net-(R16-Pad2) -> Net-(Q2-Pad3)
- R17 pad 1: Net-(C7-Pad1) -> Net-(C6-Pad1)
- R18 pad 1: Net-(C5-Pad2) -> /S_CARGA
- R18 pad 2: Net-(Q1-Pad3) -> Net-(Q3-Pad3)
- R19 pad 1: Net-(C6-Pad2) -> Net-(C7-Pad1)
- R19 pad 2: Net-(Q2-Pad3) -> Net-(R19-Pad2)
- R20 pad 1: Net-(C7-Pad2) -> /T_CARGA
- R20 pad 2: Net-(Q3-Pad3) -> Net-(Q1-Pad3)
- R21 pad 1: VAC -> /R
- R22 pad 1: VAC -> /S
- R23 pad 1: VAC -> /T
- R9 pad 2: VAC -> /R
- T1 pad 1: VAC -> /R
- T1 pad 3: Net-(D5-Pad4) -> Net-(D5-Pad3)
- T1 pad 4: Net-(D5-Pad3) -> Net-(D5-Pad4)
- U1 pad 2: +12V -> VCC
- U1 pad 3: VCC -> +12V
- U2 pad 3: Net-(U2-Pad3) -> (no net)
- U2 pad 4: Net-(Q1-Pad3) -> Net-(Q2-Pad3)
- U2 pad 5: Net-(U2-Pad5) -> (no net)
- U3 pad 3: Net-(U3-Pad3) -> (no net)
- U3 pad 4: Net-(Q2-Pad3) -> Net-(Q3-Pad3)
- U3 pad 5: Net-(U3-Pad5) -> (no net)
- U3 pad 6: Net-(R16-Pad2) -> Net-(R17-Pad2)
- U4 pad 3: Net-(U4-Pad3) -> (no net)
- U4 pad 4: Net-(Q3-Pad3) -> Net-(Q1-Pad3)
- U4 pad 5: Net-(U4-Pad5) -> (no net)
- U4 pad 6: Net-(R17-Pad2) -> Net-(R19-Pad2)
- U8 pad 10: Net-(U8-Pad10) -> (no net)
- U8 pad 11: Net-(U8-Pad11) -> (no net)
- U8 pad 12: Net-(U8-Pad12) -> (no net)
- U8 pad 17: Net-(U8-Pad17) -> (no net)
- U8 pad 18: Net-(U8-Pad18) -> (no net)
- U8 pad 19: Net-(U8-Pad19) -> (no net)
- U8 pad 20: Net-(U8-Pad20) -> (no net)
- U8 pad 21: Net-(U8-Pad21) -> (no net)
- U8 pad 22: Net-(U8-Pad22) -> (no net)
- U8 pad 24: Net-(U8-Pad24) -> (no net)
- U8 pad 32: Net-(U8-Pad32) -> (no net)
- U8 pad 4: Net-(U8-Pad4) -> (no net)
- U8 pad 5: Net-(U8-Pad5) -> (no net)
- U8 pad 7: /correnteS -> (no net)
- U8 pad 8: /correnteT -> (no net)
- U8 pad 9: Net-(U8-Pad9) -> (no net)
